File: KiCad/PPK2-USB_C-Adapter_v1.0/PPK2-USB_C-Adapter_v1.0.kicad_pcb (KiCad board)
At the start: 2 copper layers, 33.7 x 17.1 mm, 11 parts, among them J1 USB_C_Receptacle_USB2.0, J2 Conn_01x04, J3 USB_C_Receptacle_USB2.0

Commit message: last update - gerber
Parts:
- added G***: LOGO, KicadLibrary:OBJEX_Vout, F.Cu at (124.1, 85.3)
- added G***: LOGO, KicadLibrary:OBJEX_Vin, F.Cu at (121.6, 85.3)
- added G***: LOGO, KicadLibrary:OBJEX_GND, F.Cu at (126.7, 85.3)
- added G***: LOGO, KicadLibrary:OBJEX_GND, F.Cu at (119.0, 85.3)
Other:
- board text added: "Designed by Salvatore Raccardi"
- board text added: "USB-IN"
- board text added: "USB-OUT"
- board text added: "v1.0"
